File: board/bambule.kicad_pcb (KiCad board)
At the start: 2 copper layers, 55.6 x 49.2 mm, 9 parts, among them J1 Conn_01x01_Female, J2 Conn_01x01_Female, U1 AL5801

Commit message: WIP
Parts:
- added R4: 4R3 1%, Resistor_SMD:R_0805_2012Metric_Pad1.15x1.40mm_HandSolder, F.Cu at (82.0, 99.0)
- moved U1 50.2 mm to (84.0, 109.0), turned to 180 degrees
- moved R2 41.2 mm to (82.0, 105.0)
- moved R3 39.3 mm to (82.0, 102.0)
- moved R1 32.3 mm to (79.0, 96.0), turned to 90 degrees
Routing:
- net /VBUS: track 0.00 -> 24.1 mm
- net GND: track 0.00 -> 22.8 mm, vias 0 -> 1
- net Net-(R1-Pad1): track 0.00 -> 21.5 mm
- net Net-(D1-Pad1): track 0.00 -> 20.9 mm
- net Net-(R2-Pad2): track 0.00 -> 12.7 mm
- net /HEATSINK: vias 0 -> 62
- added copper zone on B.Cu, net /HEATSINK
- added copper zone on F.Cu, net /HEATSINK
Other:
- net class HEATSINK added: clearance 0.3, trace_width 0.5, via_dia 1.2, via_drill 1
- board text added: "BAMBULE v1.0"

Commit message: WIP
Parts:
- moved R1 5.00 mm to (76.0, 100.0)
Routing:
- net /VBUS: track 24.1 -> 29.9 mm
- net GND: track 22.8 -> 19.8 mm, vias 1 -> 0
- net Net-(R1-Pad1): track 21.5 -> 18.8 mm, vias 0 -> 2
Other:
- board text added: "+48V"
- board text added: "GND"
Changed lines of the file:
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@@
   (general
     (thickness 1.6)
-    (drawings 11)
-    (tracks 97)
+    (drawings 13)
+    (tracks 98)
     (zones 0)
     (modules 10)
@@
       (outputformat 1)
       (mirror false)
-      (drillshape 1)
+      (drillshape 0)
       (scaleselection 1)
-      (outputdirectory ""))
+      (outputdirectory "gerber"))
   )
   (net 0 "")
@@
   )
   (module Resistor_SMD:R_0805_2012Metric_Pad1.15x1.40mm_HandSolder (layer F.Cu)
-    (at 79 96 90)
+    (at 76 100 90)
     (descr "Resistor SMD 0805 (2012 Metric), square (rectangular) end terminal, IPC_7351 nominal with elongated pad for handsoldering. (Body size source: https://docs.google.com/spreadsheets/d/1BsfQQcO9C6DZCsRaXUlFlo91Tg2WpOkGARC1WS5S8t0/edit?usp=sharing), generated with kicad-footprint-generator")
     (tags "resistor handsolder")
@@
     )
   )
+  (gr_text GND (at 80 111 90) (layer F.SilkS)
+    (effects (font (size 1.5 1.5) (thickness 0.3)))
+  )
+  (gr_text +48V (at 80 90 90) (layer F.SilkS)
+    (effects (font (size 1.5 1.5) (thickness 0.3)))
+  )
   (gr_text "BAMBULE v1.0" (at 112 100 90) (layer F.SilkS)
     (effects (font (size 1.5 1.5) (thickness 0.3)))
@@
     (effects (font (size 3.5 2.8) (thickness 0.2)) (justify top))
   )
-  (segment (start 79 92.5) (end 94 92.5) (width 0.5) (layer F.Cu) (net 1))
-  (segment (start 75 87.5) (end 79 91.5) (width 0.5) (layer F.Cu) (net 1))
-  (segment (start 79 91.5) (end 79 92.5) (width 0.5) (layer F.Cu) (net 1))
-  (segment (start 79 94.975) (end 79 92.5) (width 0.5) (layer F.Cu) (net 1))
+  (segment (start 76 88.5) (end 75 87.5) (width 0.5) (layer F.Cu) (net 1))
+  (segment (start 94 92.5) (end 76 92.5) (width 0.5) (layer F.Cu) (net 1))
+  (segment (start 76 98.975) (end 76 92.5) (width 0.5) (layer F.Cu) (net 1))
+  (segment (start 76 92.5) (end 76 88.5) (width 0.5) (layer F.Cu) (net 1))
   (segment (start 85.9 107.5) (end 85.35 108.05) (width 0.5) (layer F.Cu) (net 2))
   (segment (start 106 107.5) (end 85.9 107.5) (width 0.5) (layer F.Cu) (net 2))
@@
   (segment (start 81.429999 109.875001) (end 81.319999 109.765001) (width 0.5) (layer F.Cu) (net 3))
   (segment (start 81.319999 107) (end 81.319999 106.144999) (width 0.5) (layer F.Cu) (net 3))
-  (via (at 81.319999 107) (size 0.8) (drill 0.4) (layers F.Cu B.Cu) (net 3))
   (segment (start 81.319999 109.765001) (end 81.319999 107) (width 0.5) (layer F.Cu) (net 3))
   (segment (start 80.975 105.8) (end 80.975 105) (width 0.5) (layer F.Cu) (net 3))
@@
   (segment (start 82.575001 109.875001) (end 81.429999 109.875001) (width 0.5) (layer F.Cu) (net 3))
   (segment (start 81.319999 106.144999) (end 80.975 105.8) (width 0.5) (layer F.Cu) (net 3))
-  (segment (start 80.754314 107) (end 81.319999 107) (width 0.5) (layer B.Cu) (net 3))
-  (segment (start 77.317398 107) (end 80.754314 107) (width 0.5) (layer B.Cu) (net 3))
-  (segment (start 75 109.317398) (end 77.317398 107) (width 0.5) (layer B.Cu) (net 3))
-  (segment (start 75 112.5) (end 75 109.317398) (width 0.5) (layer B.Cu) (net 3))
+  (segment (start 77.624999 109.875001) (end 75 112.5) (width 0.5) (layer F.Cu) (net 3))
+  (segment (start 81.429999 109.875001) (end 77.624999 109.875001) (width 0.5) (layer F.Cu) (net 3))
+  (segment (start 76 101.025) (end 76 107.5) (width 0.5) (layer F.Cu) (net 4))
+  (via (at 77 108.5) (size 0.8) (drill 0.4) (layers F.Cu B.Cu) (net 4))
+  (segment (start 76 107.5) (end 77 108.5) (width 0.5) (layer F.Cu) (net 4))
+  (segment (start 77 108.5) (end 78.5 110) (width 0.5) (layer B.Cu) (net 4))
+  (via (at 78.5 111) (size 0.8) (drill 0.4) (layers F.Cu B.Cu) (net 4))
+  (segment (start 78.5 110) (end 78.5 111) (width 0.5) (layer B.Cu) (net 4))
   (segment (start 85.35 110.775) (end 85.35 109.95) (width 0.5) (layer F.Cu) (net 4))
-  (segment (start 84.125 112) (end 85.35 110.775) (width 0.5) (layer F.Cu) (net 4))
-  (segment (start 81 112) (end 84.125 112) (width 0.5) (layer F.Cu) (net 4))
-  (segment (start 79 110) (end 81 112) (width 0.5) (layer F.Cu) (net 4))
-  (segment (start 79 97.025) (end 79 110) (width 0.5) (layer F.Cu) (net 4))
+  (segment (start 85.125 111) (end 85.35 110.775) (width 0.5) (layer F.Cu) (net 4))
+  (segment (start 78.5 111) (end 85.125 111) (width 0.5) (layer F.Cu) (net 4))
   (segment (start 83.025 99) (end 83.025 102) (width 0.5) (layer F.Cu) (net 5))
   (segment (start 83.025 102) (end 83.025 105) (width 0.5) (layer F.Cu) (net 5))
