File: board/bambule.kicad_pcb (KiCad board)
At the start: 2 copper layers, 55.6 x 49.2 mm, 10 parts, among them J1 Conn_01x01_Female, J2 Conn_01x01_Female, U1 AL5801

Commit message: WIP
Parts:
- removed R1: 430k 1%, Resistor_SMD:R_0805_2012Metric_Pad1.15x1.40mm_HandSolder
- removed R2, R3, R4: 4R3 1%, Resistor_SMD:R_0805_2012Metric_Pad1.15x1.40mm_HandSolder
- removed U1: AL5801, Package_TO_SOT_SMD:SOT-23-6_Handsoldering
- H1, H2: footprint MountingHole:MountingHole_2.5mm_Pad -> MountingHole:MountingHole_2.7mm
- J1: footprint Connector_Wire:SolderWirePad_1x01_Drill2mm -> TestPoint:TestPoint_Pad_D3.0mm
- J2: footprint Connector_Wire:SolderWirePad_1x01_Drill2mm -> TestPoint:TestPoint_Pad_D3.0mm; moved to B.Cu
- moved J1 43.8 mm to (94.0, 127.0)
- moved J2 32.5 mm to (104.1, 127.0)
Connections:
- net /VBUS renamed /VIN
- D1 pad 1: Net-(D1-Pad1) -> /GND
- J2 pad 1: GND -> /GND
Routing:
- net /VIN: track 29.9 -> 0.00 mm
- net Net-(D1-Pad1): track 20.9 -> 0.00 mm
- net GND: track 19.8 -> 0.00 mm
- net Net-(R1-Pad1): track 18.8 -> 0.00 mm, vias 2 -> 0
- net Net-(R2-Pad2): track 12.7 -> 0.00 mm
- net /HEATSINK: vias 62 -> 0
Other:
- board size 55.6 x 49.2 mm -> 55.6 x 62 mm
- board text added: "300mA"
- board text removed: "+48V"
